Commit message: test

File: alfa/my_robot_ws/src/my_robot_description/urdf/robot.urdf (robot description, URDF)
Before this commit: robot boat, 3 links, 2 joints
Links:
- added link camera_link
- added link gpu_lidar; visual cylinder length=0.05 radius=0.05
- added link odom
- link leftmotor_link: mass 5.0 -> None; geometry visual mesh filename=/home/gauss/Desktop/my_robot_ws/src/my_robot_description/mo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 scale=1 1 1
- link rightmotor_link: mass 5.0 -> None; geometry visual mesh filename=/home/gauss/Desktop/my_robot_ws/src/my_robot_description/mo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 scale=1 1 1
Joints:
- added joint camera_joint: type fixed, parent base_link, child camera_link, origin xyz=0.5 0 0.4 rpy=0 0 0
- added joint lidar_joint: type fixed, parent base_link, child gpu_lidar, origin xyz=0.5 0 0.6 rpy=0 0 0
- joint leftmotor_link_joint: axis 0 0 1 -> (none); type continuous -> fixed
- joint rightmotor_link_joint: axis 0 0 1 -> (none); type continuous -> fixed
