Commit message: bi tonla şey
algo eklendi, sdf urd düzenlendi, rviz2 düzenlendi güncel rviz ayarları eklenmeli ama

File: guncel/my_robot_ws/src/my_robot_description/urdf/robot.urdf (robot description, URDF)
Before this commit: robot boat, 5 links, 4 joints
Links:
- link base_link: geometry collision cylinder length=0.5918 radius=0.19161; visual mesh filename=package://my_robot_description/models/boat/meshes/stl/denem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 scale=1 1 1
- link leftmotor_link: geometry visual mesh filename=package://my_robot_description/models/boat/meshes/stl/denem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 scale=1 1 1
- link rightmotor_link: geometry visual mesh filename=package://my_robot_description/models/boat/meshes/stl/denem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 scale=1 1 1
